File: hardware/BaseStation/src-ext-memory/sportduino-base.kicad_pcb (KiCad board)
At the start: 2 copper layers, 71.1 x 30.5 mm, 45 parts, among them X1 Battery, X2 Prog, X3 RC522

Commit message: Updated v3m PCB
Parts:
- removed BZ1*: PinHeader_1x01_P2.54mm_Vertical, Connector_PinHeader_2.54mm:PinHeader_1x01_P2.54mm_Vertical
- removed TP6: TestPoint, TestPoint:TestPoint_THTPad_D1.5mm_Drill0.7mm
- removed VD2A*, VD2B*: D_SMA, Diode_SMD:D_SMA
- added SW1: SW_Reed, Button_Switch_THT:SW_reed, F.Cu at (167.0, 112.4)
- BZ1: footprint Buzzer_Beeper:Buzzer_12x9.5RM7.6 -> Buzzer_Beeper:MagneticBuzzer_ProSignal_ABT-410-RC
- moved X2 89.1 mm to (197.5, 89.5), turned to 0 degrees
- moved D4 46.6 mm to (169.9, 85.1)
- moved C1 42.1 mm to (178.8, 104.3), turned to 270 degrees
- moved R7 38.6 mm to (173.5, 105.9), turned to 0 degrees
- moved C3 36.6 mm to (130.5, 91.4), turned to 180 degrees
- moved VT1 34.7 mm to (138.8, 111.5), turned to 180 degrees
- moved D1 34.7 mm to (130.6, 86.9), turned to 90 degrees
- moved R11 34.3 mm to (191.8, 74.4)
- moved C8 34.2 mm to (191.8, 77.0), turned to 0 degrees
- moved D3 32.6 mm to (182.9, 74.9), turned to 180 degrees
- moved C2 32.0 mm to (130.6, 82.5), turned to 180 degrees
- moved VD2 31.7 mm to (138.2, 72.6)
- moved C9 30.3 mm to (175.3, 75.7), turned to 90 degrees
- moved R9 30.2 mm to (143.8, 73.9)
- moved R4 29.6 mm to (147.7, 111.5), turned to 90 degrees
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Connections:
- D2 pad 12: Net-(D2-Pad12) -> /PB0
- D2 pad 26: /VCCR -> PC3
- JP1 pad 3: /VCCR -> PC3
- JP2 pad 3: /VCCR -> PC3
- TP3 pad 1: Net-(D2-Pad12) -> PC3
- X2 pad 2: +BATT -> +3V3
- X2 pad 3: +3V3 -> PC3
- X3 pad 5: PD6 -> /PB0
Routing:
- net GNDD: track 234.4 -> 126.1 mm, vias 7 -> 3
- net PB4: track 92.9 -> 19.0 mm
- net PB3: track 92.5 -> 21.3 mm
- net +BATT: track 103.3 -> 35.7 mm
- net PC3: track 0.00 -> 56.1 mm, vias 0 -> 1
- net PB5: track 73.9 -> 27.1 mm
- net ADCIN: track 9.75 -> 47.9 mm, vias 0 -> 2
- net Net-(BZ1-Pad2): track 45.8 -> 9.75 mm
- net ADCEN: track 7.98 -> 42.5 mm, vias 0 -> 2
- net Net-(C7-Pad1): track 56.3 -> 25.0 mm, vias 2 -> 0
- net Net-(VD2-Pad3): track 29.4 -> 0.00 mm
- net /BUZ: track 3.75 -> 32.8 mm, vias 0 -> 2
- net RST: track 5.33 -> 28.9 mm
- net Net-(D2-Pad12): track 19.9 -> 0.00 mm, vias 1 -> 0
- net Net-(C8-Pad1): track 9.32 -> 29.1 mm, vias 0 -> 2
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- removed copper zone on B.Cu, net GNDD
- removed copper zone on F.Cu, net GNDD
Other:
- board size 71.1 x 30.5 mm -> 76.8 x 45.7 mm
- net class Default: trace_width 0.3 -> 0.5
- net class power: trace_width 0.5 -> 0.6

Commit message: Updated PCB
Parts:
- added G***: LOGO, src-ext-memory:logo, F.Cu at (182.1, 80.8)
- D3: value DS3231SN -> (none)
- moved VT1 78.0 mm to (198.2, 60.9), turned to 0 degrees
- moved C3 76.7 mm to (206.5, 81.0), turned to 0 degrees
- moved C2 76.3 mm to (206.5, 89.9), turned to 0 degrees
- moved D1 75.9 mm to (206.5, 85.6), turned to 270 degrees
- moved BZ1 74.9 mm to (204.3, 75.3), turned to 90 degrees
- moved X1 74.4 mm to (205.0, 93.7), turned to 90 degrees
- moved R5 69.9 mm to (192.6, 60.9), turned to 90 degrees
- moved VD2 66.5 mm to (198.9, 99.8), turned to 270 degrees
- moved R4 65.5 mm to (189.3, 60.9), turned to 270 degrees
- moved VD1 63.1 mm to (138.0, 94.3), turned to 90 degrees
- moved JP3 62.9 mm to (198.9, 94.5), turned to 180 degrees
- moved X2 58.3 mm to (139.6, 82.9), turned to 180 degrees
- moved X3 55.5 mm to (144.6, 72.1), turned to 0 degrees
- moved R9 55.3 mm to (193.3, 98.5), turned to 0 degrees
- moved SW1 52.4 mm to (170.0, 60.0), turned to 0 degrees
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Routing:
- net GNDD: track 126.1 -> 253.1 mm, vias 3 -> 7
- net TX: track 33.2 -> 69.9 mm, vias 2 -> 0
- net +3V3: track 190.1 -> 226.1 mm
- net RX: track 41.6 -> 63.1 mm, vias 1 -> 0
- net ADCIN: track 47.9 -> 69.2 mm
- net Net-(C7-Pad1): track 25.0 -> 32.7 mm
- net Net-(C1-Pad2): track 33.4 -> 39.1 mm, vias 0 -> 1
- net PD6: track 27.4 -> 31.9 mm
- net RST: track 28.9 -> 32.8 mm, vias 0 -> 2
- net 32K: track 31.0 -> 33.3 mm
- net Net-(D2-Pad11): track 17.8 -> 19.0 mm
- net Net-(BZ1-Pad2): track 9.75 -> 10.4 mm
- net Net-(D2-Pad32): track 25.2 -> 25.8 mm
- added copper zone on B.Cu, net GNDD
- added copper zone on F.Cu, net GNDD
Other:
- outline, holes or cut-outs redrawn
- net class power: trace_width 0.6 -> 0.8
- board text added: "+"
- board text added: "v3 2019-12-12"
