File: hardware/BaseStation/src/sportiduino-base.kicad_pcb (KiCad board)
At the start: 2 copper layers, 73 x 45 mm, 46 parts, among them SW1 SW_Reed, X1 Battery, X2 Prog, X3 RC522, X4 MINI RC522, X5 Charge

Commit message: PCB: desc pos fix
Parts:
- TP1, TP2, TP4, TP5: value TestPoint -> (none)
- VD2, VD3: value 0805 -> (none)
