File: hardware/BaseStation/src-v4/sportiduino-base-v4.kicad_sch (KiCad schematic)
At the start: 43 parts, among them SW1 SW_Reed, X1 Battery, X2 Prog, X4 MINI RC522, X5 Charge

Commit message: New PCB (wip)
Parts:
- removed TP1, TP2, TP4, TP5: TestPoint, TestPoint:TestPoint_THTPad_D1.5mm_Drill0.7mm, symbol Connector:TestPoint
- C1, C10, C4, C5, C6, C7, C9: footprint Capacitor_SMD:C_0805_2012Metric_Pad1.15x1.40mm_HandSolder -> Capacitor_SMD:C_0603_1608Metric_Pad1.08x0.95mm_HandSolder
- R1, R10, R11, R2, R3, R4, R5, R6, R8, R9: footprint Resistor_SMD:R_0805_2012Metric_Pad1.15x1.40mm_HandSolder -> Resistor_SMD:R_0603_1608Metric_Pad0.98x0.95mm_HandSolder
- R12, R13, R14: footprint Resistor_SMD:R_0805_2012Metric_Pad1.20x1.40mm_HandSolder -> Resistor_SMD:R_0603_1608Metric_Pad0.98x0.95mm_HandSolder
- VD1: footprint LED_THT:LED_D3.0mm -> LED_SMD:LED_1210_3225Metric_Pad1.42x2.65mm_HandSolder
- X1: footprint Connector_JST:JST_XH_B2B-XH-A_1x02_P2.50mm_Vertical -> Connector_JST:JST_ZH_B2B-ZR_1x02_P1.50mm_Vertical
- X2: footprint Connector_IDC:IDC-Header_2x05_P2.54mm_Vertical -> Connector_Hirose:Hirose_DF13-10P-1.25DSA_1x10_P1.25mm_Vertical
- X5: footprint Connector_PinHeader_2.54mm:PinHeader_1x02_P2.54mm_Vertical -> Connector_JST:JST_PH_B2B-PH-K_1x02_P2.00mm_Vertical
- renumbered X4 to X3
Connections:
- no-connect marks 0 -> 4
