File: hardware/BaseStation/src-v3bm/sportiduino-base-v3bm.kicad_sch (KiCad schematic)
At the start: 39 parts, among them SW1 SW_Reed, X1 Battery, X2 Prog, X3 MINI RC522, X5 Charge

Commit message: pcb v3bm update
Parts:
- R14: value 3K3 -> 2K4
Changed lines of the file:
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@@
 			)
 		)
-		(property "Value" "3K3"
+		(property "Value" "2K4"
 			(at 150.368 187.833 0)
 			(effects
